File: pcb/airsticks_pcb.kicad_sch (KiCad schematic)
At the start: 17 parts, among them J1 USB_C_Receptacle_USB2.0, J2 STM_LINK, J3 USB_SERIAL_TTL, J4 I2C, J5 AudioJack3, U1 STM32G441KBT6, U4 PAM8302AAS, U5 TC1262-33

Commit message: pcb ready for printing
Parts:
- removed C2: 0.1uF, Capacitor_SMD:C_0805_2012Metric_Pad1.18x1.45mm_HandSolder, symbol Device:C
Connections:
- net AUDIO+: now also U1.9 (PA4)
- net at C1.2, U4.3 (IN+): now also U4.4 (IN-)
- no-connect marks 45 -> 44
Other:
- moved on the sheet: C1
Changed lines of the file:
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@@
   (junction (at 106.68 30.48) (diameter 0) (color 0 0 0 0)
+  )
+  (junction (at 113.03 135.89) (diameter 0) (color 0 0 0 0)
   )
   (junction (at 86.36 59.69) (diameter 0) (color 0 0 0 0)
@@
   (no_connect (at 241.3 109.22))
   (no_connect (at 138.43 73.66))
-  (no_connect (at 26.67 41.91))
   (no_connect (at 82.55 36.83))
   (no_connect (at 138.43 30.48))
@@
     (stroke (width 0) (type default) (color 0 0 0 0))
   )
-  (wire (pts (xy 92.71 140.97) (xy 105.41 140.97))
-    (stroke (width 0) (type default) (color 0 0 0 0))
-  )
   (wire (pts (xy 109.22 127) (xy 109.22 128.27))
     (stroke (width 0) (type default) (color 0 0 0 0))
@@
     (stroke (width 0) (type default) (color 0 0 0 0))
   )
-  (wire (pts (xy 92.71 135.89) (xy 105.41 135.89))
+  (wire (pts (xy 92.71 135.89) (xy 104.14 135.89))
     (stroke (width 0) (type default) (color 0 0 0 0))
   )
@@
     (stroke (width 0) (type default) (color 0 0 0 0))
   )
+  (wire (pts (xy 22.86 41.91) (xy 26.67 41.91))
+    (stroke (width 0) (type default) (color 0 0 0 0))
+  )
   (wire (pts (xy 247.65 31.75) (xy 252.73 31.75))
     (stroke (width 0) (type default) (color 0 0 0 0))
@@
     (stroke (width 0) (type default) (color 0 0 0 0))
   )
+  (wire (pts (xy 111.76 135.89) (xy 113.03 135.89))
+    (stroke (width 0) (type default) (color 0 0 0 0))
+  )
   (wire (pts (xy 219.71 109.22) (xy 224.79 109.22))
     (stroke (width 0) (type default) (color 0 0 0 0))
@@
   )
   (wire (pts (xy 86.36 59.69) (xy 82.55 59.69))
+    (stroke (width 0) (type default) (color 0 0 0 0))
+  )
+  (wire (pts (xy 113.03 135.89) (xy 113.03 140.97))
     (stroke (width 0) (type default) (color 0 0 0 0))
   )
@@
     (effects (font (size 1.27 1.27)) (justify right bottom))
   )
+  (label "AUDIO+" (at 22.86 41.91 180)
+    (effects (font (size 1.27 1.27)) (justify right bottom))
+  )
   (label "SWCLK" (at 246.38 69.85 180)
     (effects (font (size 1.27 1.27)) (justify right bottom))
-  )
-  (label "AUDIO-" (at 92.71 140.97 0)
-    (effects (font (size 1.27 1.27)) (justify left bottom))
   )
   (label "I2C1_SDA" (at 105.41 83.82 180)
@@
     (pin "1")
   )
-  (symbol (lib_id "Device:C") (at 109.22 135.89 90) (unit 1)
-    (in_bom yes) (on_board yes)
-    (property "Reference" "C1" (id 0) (at 113.03 134.62 90)
-      (effects (font (size 1.27 1.27)) (justify left))
-    )
-    (property "Value" "0.1uF" (id 1) (at 107.95 134.62 90)
-      (effects (font (size 1.27 1.27)) (justify left))
-    )
-    (property "Footprint" "Capacitor_SMD:C_0805_2012Metric_Pad1.18x1.45mm_HandSolder" (id 2) (at 113.03 134.9248 0)
-      (effects (font (size 1.27 1.27)) hide)
-    )
-    (property "Datasheet" "~" (id 3) (at 109.22 135.89 0)
+  (symbol (lib_id "Device:C") (at 107.95 135.89 90) (unit 1)
+    (in_bom yes) (on_board yes)
+    (property "Reference" "C1" (id 0) (at 111.76 134.62 90)
+      (effects (font (size 1.27 1.27)) (justify left))
+    )
+    (property "Value" "0.1uF" (id 1) (at 106.68 134.62 90)
+      (effects (font (size 1.27 1.27)) (justify left))
+    )
+    (property "Footprint" "Capacitor_SMD:C_0805_2012Metric_Pad1.18x1.45mm_HandSolder" (id 2) (at 111.76 134.9248 0)
+      (effects (font (size 1.27 1.27)) hide)
+    )
+    (property "Datasheet" "~" (id 3) (at 107.95 135.89 0)
       (effects (font (size 1.27 1.27)) hide)
     )
@@
     )
     (pin "1")
-  )
-  (symbol (lib_id "Device:C") (at 109.22 140.97 90) (unit 1)
-    (in_bom yes) (on_board yes)
-    (property "Reference" "C2" (id 0) (at 113.03 139.7 90)
-      (effects (font (size 1.27 1.27)) (justify left))
-    )
-    (property "Value" "0.1uF" (id 1) (at 107.95 139.7 90)
-      (effects (font (size 1.27 1.27)) (justify left))
-    )
-    (property "Footprint" "Capacitor_SMD:C_0805_2012Metric_Pad1.18x1.45mm_HandSolder" (id 2) (at 113.03 140.0048 0)
-      (effects (font (size 1.27 1.27)) hide)
-    )
-    (property "Datasheet" "~" (id 3) (at 109.22 140.97 0)
-      (effects (font (size 1.27 1.27)) hide)
-    )
-    (pin "1")
-    (pin "2")
   )
   (symbol (lib_id "power:GND") (at 86.36 71.12 0) (unit 1)
@@
       (reference "C1") (unit 1) (value "0.1uF") (footprint "Capacitor_SMD:C_0805_2012Metric_Pad1.18x1.45mm_HandSolder")
     )
-    (path "/81565611-678b-4f51-b84b-d6ed83ca9978"
-      (reference "C2") (unit 1) (value "0.1uF") (footprint "Capacitor_SMD:C_0805_2012Metric_Pad1.18x1.45mm_HandSolder")
-    )
     (path "/b1deaa6f-a2c3-48dc-8451-43d1195f4686"

Commit message: updated PCB to reflect changes we made. NOTE: still need to make the boot0 change, as it is still currently floating
Connections:
- net SCL is gone; now on net I2C_SCL: J4.2 (Pin_2)
- net SDA is gone; now on net I2C_SDA: J4.1 (Pin_1)
- net GND: no longer J1.S1 (SHIELD)
- net RX: now also U1.8 (PA3)
- net SWCLK: now also U1.24 (PA14)
- net SWDIO: now also U1.23 (PA13)
- net TX: now also U1.7 (PA2)
- net I2C_SCL: now reaches U1.25 (PA15)
- net I2C_SCL: now also xlr_left1.13 (SCL), xlr_right1.13 (SCL)
- net I2C_SDA: now reaches U1.30 (PB7)
- net I2C_SDA: now also xlr_left1.14 (SDA), xlr_right1.14 (SDA)
- removed net I2C1_SDA: U1.24 (PA14), xlr_left1.14 (SDA), xlr_right1.14 (SDA)
- removed net I2C1_SLC: U1.23 (PA13), xlr_left1.13 (SCL), xlr_right1.13 (SCL)
- no-connect marks 44 -> 41
Changed lines of the file:
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@@
   (no_connect (at 190.5 44.45))
   (no_connect (at 26.67 59.69))
-  (no_connect (at 82.55 41.91))
   (no_connect (at 190.5 36.83))
   (no_connect (at 190.5 52.07))
+  (no_connect (at 167.64 69.85))
   (no_connect (at 243.84 77.47))
   (no_connect (at 223.52 74.93))
@@
   (no_connect (at 26.67 34.29))
   (no_connect (at 26.67 31.75))
-  (no_connect (at 26.67 39.37))
-  (no_connect (at 26.67 36.83))
   (no_connect (at 243.84 74.93))
-  (no_connect (at 26.67 69.85))
   (no_connect (at 26.67 52.07))
   (no_connect (at 241.3 109.22))
@@
     (stroke (width 0) (type default) (color 0 0 0 0))
   )
-  (wire (pts (xy 167.64 71.12) (xy 167.64 69.85))
+  (wire (pts (xy 85.09 41.91) (xy 82.55 41.91))
     (stroke (width 0) (type default) (color 0 0 0 0))
   )
@@
     (stroke (width 0) (type default) (color 0 0 0 0))
   )
-  (wire (pts (xy 219.71 104.14) (xy 224.79 104.14))
+  (wire (pts (xy 217.17 104.14) (xy 224.79 104.14))
     (stroke (width 0) (type default) (color 0 0 0 0))
   )
@@
     (stroke (width 0) (type default) (color 0 0 0 0))
   )
-  (wire (pts (xy 167.64 71.12) (xy 175.26 71.12))
-    (stroke (width 0) (type default) (color 0 0 0 0))
-  )
   (wire (pts (xy 219.71 73.66) (xy 219.71 72.39))
     (stroke (width 0) (type default) (color 0 0 0 0))
@@
     (stroke (width 0) (type default) (color 0 0 0 0))
   )
+  (wire (pts (xy 22.86 67.31) (xy 26.67 67.31))
+    (stroke (width 0) (type default) (color 0 0 0 0))
+  )
   (wire (pts (xy 119.38 127) (xy 123.19 127))
     (stroke (width 0) (type default) (color 0 0 0 0))
   )
-  (wire (pts (xy 219.71 106.68) (xy 224.79 106.68))
+  (wire (pts (xy 217.17 106.68) (xy 224.79 106.68))
     (stroke (width 0) (type default) (color 0 0 0 0))
   )
@@
     (stroke (width 0) (type default) (color 0 0 0 0))
   )
-  (wire (pts (xy 22.86 67.31) (xy 26.67 67.31))
-    (stroke (width 0) (type default) (color 0 0 0 0))
-  )
   (wire (pts (xy 107.95 76.2) (xy 106.68 76.2))
     (stroke (width 0) (type default) (color 0 0 0 0))
@@
     (stroke (width 0) (type default) (color 0 0 0 0))
   )
+  (wire (pts (xy 22.86 69.85) (xy 26.67 69.85))
+    (stroke (width 0) (type default) (color 0 0 0 0))
+  )
   (wire (pts (xy 175.26 71.12) (xy 182.88 71.12))
     (stroke (width 0) (type default) (color 0 0 0 0))
@@
     (stroke (width 0) (type default) (color 0 0 0 0))
   )
+  (wire (pts (xy 22.86 36.83) (xy 26.67 36.83))
+    (stroke (width 0) (type default) (color 0 0 0 0))
+  )
   (wire (pts (xy 219.71 72.39) (xy 227.33 72.39))
     (stroke (width 0) (type default) (color 0 0 0 0))
@@
     (stroke (width 0) (type default) (color 0 0 0 0))
   )
+  (wire (pts (xy 22.86 39.37) (xy 26.67 39.37))
+    (stroke (width 0) (type default) (color 0 0 0 0))
+  )
   (wire (pts (xy 105.41 88.9) (xy 107.95 88.9))
     (stroke (width 0) (type default) (color 0 0 0 0))
@@
     (stroke (width 0) (type default) (color 0 0 0 0))
   )
-  (label "I2C1_SLC" (at 105.41 43.18 180)
-    (effects (font (size 1.27 1.27)) (justify right bottom))
-  )
-  (label "I2C1_SDA" (at 105.41 40.64 180)
+  (label "RX" (at 22.86 39.37 180)
+    (effects (font (size 1.27 1.27)) (justify right bottom))
+  )
+  (label "I2C_SCL" (at 105.41 43.18 180)
+    (effects (font (size 1.27 1.27)) (justify right bottom))
+  )
+  (label "I2C_SDA" (at 105.41 40.64 180)
     (effects (font (size 1.27 1.27)) (justify right bottom))
   )
@@
     (effects (font (size 1.27 1.27)) (justify right bottom))
   )
-  (label "I2C1_SDA" (at 105.41 83.82 180)
-    (effects (font (size 1.27 1.27)) (justify right bottom))
-  )
-  (label "I2C1_SDA" (at 22.86 67.31 180)
+  (label "I2C_SDA" (at 105.41 83.82 180)
     (effects (font (size 1.27 1.27)) (justify right bottom))
   )
@@
     (effects (font (size 1.27 1.27)) (justify right bottom))
   )
-  (label "I2C1_SLC" (at 105.41 86.36 180)
+  (label "I2C_SCL" (at 105.41 86.36 180)
     (effects (font (size 1.27 1.27)) (justify right bottom))
   )
@@
     (effects (font (size 1.27 1.27)) (justify left bottom))
   )
+  (label "SWCLK" (at 22.86 67.31 180)
+    (effects (font (size 1.27 1.27)) (justify right bottom))
+  )
   (label "AUDIO+" (at 92.71 135.89 0)
     (effects (font (size 1.27 1.27)) (justify left bottom))
@@
     (effects (font (size 1.27 1.27)) (justify left bottom))
   )
+  (label "SWDIO" (at 22.86 64.77 180)
+    (effects (font (size 1.27 1.27)) (justify right bottom))
+  )
   (label "SWDIO" (at 246.38 67.31 180)
     (effects (font (size 1.27 1.27)) (justify right bottom))
   )
-  (label "I2C1_SLC" (at 22.86 64.77 180)
-    (effects (font (size 1.27 1.27)) (justify right bottom))
-  )
   (label "+3V3" (at 105.41 88.9 180)
     (effects (font (size 1.27 1.27)) (justify right bottom))
@@
     (effects (font (size 1.27 1.27)) (justify left bottom))
   )
-  (label "SCL" (at 219.71 106.68 0)
-    (effects (font (size 1.27 1.27)) (justify left bottom))
-  )
-  (label "SDA" (at 219.71 104.14 0)
+  (label "TX" (at 22.86 36.83 180)
+    (effects (font (size 1.27 1.27)) (justify right bottom))
+  )
+  (label "I2C_SDA" (at 85.09 41.91 0)
+    (effects (font (size 1.27 1.27)) (justify left bottom))
+  )
+  (label "I2C_SCL" (at 217.17 106.68 0)
+    (effects (font (size 1.27 1.27)) (justify left bottom))
+  )
+  (label "I2C_SDA" (at 217.17 104.14 0)
     (effects (font (size 1.27 1.27)) (justify left bottom))
   )
@@
     (effects (font (size 1.27 1.27)) (justify left bottom))
   )
+  (label "I2C_SCL" (at 22.86 69.85 180)
+    (effects (font (size 1.27 1.27)) (justify right bottom))
+  )
   (label "ACC_INT1" (at 85.09 31.75 0)
